Commit message: fix urdf

File: packages/physicalai-lekiwi-plugin/urdf/lekiwi/urdf/LeKiwi.urdf (robot description, URDF)
Before this commit: robot LeKiwi, 11 links, 10 joints
Links:
- removed link arm_base
- removed link back_wheel_link
- removed link base_link
- removed link elbow_flex_link
- removed link gripper_link
- removed link left_wheel_link
- removed link right_wheel_link
- removed link shoulder_lift_link
- removed link shoulder_pan_link
- removed link wrist_flex_link
- removed link wrist_roll_link
- added link 4-Omni-Directional-Wheel_Single_Body-v1, mass 1.3542854082324305; collision mesh filename=meshes/4-Omni-Directional-Wheel_Single_Body-v1.stl scale=0.001 0.001 0.001; visual mesh filename=meshes/4-Omni-Directional-Wheel_Single_Body-v1.stl scale=0.001 0.001 0.001
- added link 4-Omni-Directional-Wheel_Single_Body-v1-1, mass 1.3542854082324305; collision mesh filename=meshes/4-Omni-Directional-Wheel_Single_Body-v1-1.stl scale=0.001 0.001 0.001; visual mesh filename=meshes/4-Omni-Directional-Wheel_Single_Body-v1-1.stl scale=0.001 0.001 0.001
- added link 4-Omni-Directional-Wheel_Single_Body-v1-2, mass 1.3542854082324305; collision mesh filename=meshes/4-Omni-Directional-Wheel_Single_Body-v1-2.stl scale=0.001 0.001 0.001; visual mesh filename=meshes/4-Omni-Directional-Wheel_Single_Body-v1-2.stl scale=0.001 0.001 0.001
- added link 94868A713_NO-THREADS_Female-Threaded-Hex-Standoff, mass 0.006150070863406618; collision mesh filename=meshes/94868A713_NO-THREADS_Female-Threaded-Hex-Standoff.stl scale=0.001 0.001 0.001; visual mesh filename=meshes/94868A713_NO-THREADS_Female-Threaded-Hex-Standoff.stl scale=0.001 0.001 0.001
- added link 94868A713_NO-THREADS_Female-Threaded-Hex-Standoff-1, mass 0.006150070863406618; collision mesh filename=meshes/94868A713_NO-THREADS_Female-Threaded-Hex-Standoff-1.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 scale=0.001 0.001 0.001; visual mesh filename=meshes/94868A713_NO-THREADS_Female-Threaded-Hex-Standoff-1.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 scale=0.001 0.001 0.001
- added link 94868A713_NO-THREADS_Female-Threaded-Hex-Standoff-2, mass 0.006150070863406618; collision mesh filename=meshes/94868A713_NO-THREADS_Female-Threaded-Hex-Standoff-2.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 scale=0.001 0.001 0.001; visual mesh filename=meshes/94868A713_NO-THREADS_Female-Threaded-Hex-Standoff-2.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 scale=0.001 0.001 0.001
- added link 94868A713_NO-THREADS_Female-Threaded-Hex-Standoff-3, mass 0.006150070863406618; collision mesh filename=meshes/94868A713_NO-THREADS_Female-Threaded-Hex-Standoff-3.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 scale=0.001 0.001 0.001; visual mesh filename=meshes/94868A713_NO-THREADS_Female-Threaded-Hex-Standoff-3.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 scale=0.001 0.001 0.001
- added link 94868A713_NO-THREADS_Female-Threaded-Hex-Standoff-4, mass 0.006150070863406618; collision mesh filename=meshes/94868A713_NO-THREADS_Female-Threaded-Hex-Standoff-4.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 scale=0.001 0.001 0.001; visual mesh filename=meshes/94868A713_NO-THREADS_Female-Threaded-Hex-Standoff-4.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 scale=0.001 0.001 0.001
- added link 94868A713_NO-THREADS_Female-Threaded-Hex-Standoff-5, mass 0.006150070863406618; collision mesh filename=meshes/94868A713_NO-THREADS_Female-Threaded-Hex-Standoff-5.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 scale=0.001 0.001 0.001; visual mesh filename=meshes/94868A713_NO-THREADS_Female-Threaded-Hex-Standoff-5.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 scale=0.001 0.001 0.001
- added link Base_08q-v1, mass 1.2829039880853146; collision mesh filename=meshes/Base_08q-v1.stl scale=0.001 0.001 0.001; visual mesh filename=meshes/Base_08q-v1.stl scale=0.001 0.001 0.001
- added link Battery---Battery-5.2-Ah-DC5521-Plug-v2, mass 1.2215469988184764; collision mesh filename=meshes/Battery---Battery-5.2-Ah-DC5521-Plug-v2.stl scale=0.001 0.001 0.001; visual mesh filename=meshes/Battery---Battery-5.2-Ah-DC5521-Plug-v2.stl scale=0.001 0.001 0.001
- added link Bottom-V2-v3, mass 0.14588862570926195; collision mesh filename=meshes/Bottom-V2-v3.stl scale=0.001 0.001 0.001; visual mesh filename=meshes/Bottom-V2-v3.stl scale=0.001 0.001 0.001
- added link Camera-Model-v3, mass 0.039920058315088616; collision mesh filename=meshes/Camera-Model-v3.stl scale=0.001 0.001 0.001; visual mesh filename=meshes/Camera-Model-v3.stl scale=0.001 0.001 0.001
- added link Camera-Model-v3-1, mass 0.039920058315088616; collision mesh filename=meshes/Camera-Model-v3-1.stl scale=0.001 0.001 0.001; visual mesh filename=meshes/Camera-Model-v3-1.stl scale=0.001 0.001 0.001
- added link Camera-Mount-v8, mass 0.09265469509875414; collision mesh filename=meshes/Camera-Mount-v8.stl scale=0.001 0.001 0.001; visual mesh filename=meshes/Camera-Mount-v8.stl scale=0.001 0.001 0.001
- added link Moving_Jaw_08d-v1, mass 0.1586808414280307; collision mesh filename=meshes/Moving_Jaw_08d-v1.stl scale=0.001 0.001 0.001; visual mesh filename=meshes/Moving_Jaw_08d-v1.stl scale=0.001 0.001 0.001
- added link Passive_Horn_01-v1, mass 0.00454511487954422; collision mesh filename=meshes/Passive_Horn_01-v1.stl scale=0.001 0.001 0.001; visual mesh filename=meshes/Passive_Horn_01-v1.stl scale=0.001 0.001 0.001
- added link Rotation_Pitch_08i-v1, mass 0.5385469320676795; collision mesh filename=meshes/Rotation_Pitch_08i-v1.stl scale=0.001 0.001 0.001; visual mesh filename=meshes/Rotation_Pitch_08i-v1.stl scale=0.001 0.001 0.001
- added link SO_ARM100_08k_116_Square-v1, mass 0.9906249126045027; collision mesh filename=meshes/SO_ARM100_08k_116_Square-v1.stl scale=0.001 0.001 0.001; visual mesh filename=meshes/SO_ARM100_08k_116_Square-v1.stl scale=0.001 0.001 0.001
- added link SO_ARM100_08k_Asym_Mirror_Clip-v1, mass 0.10853073755546007; collision mesh filename=meshes/SO_ARM100_08k_Asym_Mirror_Clip-v1.stl scale=0.001 0.001 0.001; visual mesh filename=meshes/SO_ARM100_08k_Asym_Mirror_Clip-v1.stl scale=0.001 0.001 0.001
- added link SO_ARM100_08k_Mirror-v1, mass 0.8772447501056027; collision mesh filename=meshes/SO_ARM100_08k_Mirror-v1.stl scale=0.001 0.001 0.001; visual mesh filename=meshes/SO_ARM100_08k_Mirror-v1.stl scale=0.001 0.001 0.001
- added link ST3215_Servo_Motor-v1, mass 0.0658962961901927; collision mesh filename=meshes/ST3215_Servo_Motor-v1.stl scale=0.001 0.001 0.001; visual mesh filename=meshes/ST3215_Servo_Motor-v1.stl scale=0.001 0.001 0.001
- added link ST3215_Servo_Motor-v1-1, mass 0.0658962961901927; collision mesh filename=meshes/ST3215_Servo_Motor-v1-1.stl scale=0.001 0.001 0.001; visual mesh filename=meshes/ST3215_Servo_Motor-v1-1.stl scale=0.001 0.001 0.001
- added link ST3215_Servo_Motor-v1-2, mass 0.0658962961901927; collision mesh filename=meshes/ST3215_Servo_Motor-v1-2.stl scale=0.001 0.001 0.001; visual mesh filename=meshes/ST3215_Servo_Motor-v1-2.stl scale=0.001 0.001 0.001
- added link STS3215_03a-v1, mass 0.2843033831904074; collision mesh filename=meshes/STS3215_03a-v1.stl scale=0.001 0.001 0.001; visual mesh filename=meshes/STS3215_03a-v1.stl scale=0.001 0.001 0.001
- added link STS3215_03a-v1-1, mass 0.2843033831904074; collision mesh filename=meshes/STS3215_03a-v1-1.stl scale=0.001 0.001 0.001; visual mesh filename=meshes/STS3215_03a-v1-1.stl scale=0.001 0.001 0.001
- added link STS3215_03a-v1-2, mass 0.2843033831904074; collision mesh filename=meshes/STS3215_03a-v1-2.stl scale=0.001 0.001 0.001; visual mesh filename=meshes/STS3215_03a-v1-2.stl scale=0.001 0.001 0.001
- added link STS3215_03a-v1-3, mass 0.2843033831904074; collision mesh filename=meshes/STS3215_03a-v1-3.stl scale=0.001 0.001 0.001; visual mesh filename=meshes/STS3215_03a-v1-3.stl scale=0.001 0.001 0.001
- added link STS3215_03a-v1-4, mass 0.2843033831904074; collision mesh filename=meshes/STS3215_03a-v1-4.stl scale=0.001 0.001 0.001; visual mesh filename=meshes/STS3215_03a-v1-4.stl scale=0.001 0.001 0.001
- added link STS3215_03a_Wrist_Roll-v1, mass 0.2799142523131049; collision mesh filename=meshes/STS3215_03a_Wrist_Roll-v1.stl scale=0.001 0.001 0.001; visual mesh filename=meshes/STS3215_03a_Wrist_Roll-v1.stl scale=0.001 0.001 0.001
- added link Top-V2-v2, mass 0.1256590419653392; collision mesh filename=meshes/Top-V2-v2.stl scale=0.001 0.001 0.001; visual mesh filename=meshes/Top-V2-v2.stl scale=0.001 0.001 0.001
- added link WaveShare_Mounting_Plate_01d-v1, mass 0.07141322001638221; collision mesh filename=meshes/WaveShare_Mounting_Plate_01d-v1.stl scale=0.001 0.001 0.001; visual mesh filename=meshes/WaveShare_Mounting_Plate_01d-v1.stl scale=0.001 0.001 0.001
- added link Wrist-Camera-Mount-v11, mass 0.14254654385043797; collision mesh filename=meshes/Wrist-Camera-Mount-v11.stl scale=0.001 0.001 0.001; visual mesh filename=meshes/Wrist-Camera-Mount-v11.stl scale=0.001 0.001 0.001
- added link Wrist_Roll_08c-v1, mass 0.44698022927880193; collision mesh filename=meshes/Wrist_Roll_08c-v1.stl scale=0.001 0.001 0.001; visual mesh filename=meshes/Wrist_Roll_08c-v1.stl scale=0.001 0.001 0.001
- added link Wrist_Roll_Pitch_08i-v1, mass 0.2392168278135931; collision mesh filename=meshes/Wrist_Roll_Pitch_08i-v1.stl scale=0.001 0.001 0.001; visual mesh filename=meshes/Wrist_Roll_Pitch_08i-v1.stl scale=0.001 0.001 0.001
- added link base_plate_layer1-v5, mass 1.9468624348344596; collision mesh filename=meshes/base_plate_layer1-v5.stl scale=0.001 0.001 0.001; visual mesh filename=meshes/base_plate_layer1-v5.stl scale=0.001 0.001 0.001
- added link base_plate_layer2-v3, mass 1.9153836917607525; collision mesh filename=meshes/base_plate_layer2-v3.stl scale=0.001 0.001 0.001; visual mesh filename=meshes/base_plate_layer2-v3.stl scale=0.001 0.001 0.001
- added link drive_motor_mount-v11, mass 0.047242276734470956; collision mesh filename=meshes/drive_motor_mount-v11.stl scale=0.001 0.001 0.001; visual mesh filename=meshes/drive_motor_mount-v11.stl scale=0.001 0.001 0.001
- added link drive_motor_mount-v11-1, mass 0.047242276734470956; collision mesh filename=meshes/drive_motor_mount-v11-1.stl scale=0.001 0.001 0.001; visual mesh filename=meshes/drive_motor_mount-v11-1.stl scale=0.001 0.001 0.001
- added link drive_motor_mount-v11-2, mass 0.047242276734470956; collision mesh filename=meshes/drive_motor_mount-v11-2.stl scale=0.001 0.001 0.001; visual mesh filename=meshes/drive_motor_mount-v11-2.stl scale=0.001 0.001 0.001
- added link lipo_battery_mount-v3, mass 0.2984320446179905; collision mesh filename=meshes/lipo_battery_mount-v3.stl scale=0.001 0.001 0.001; visual mesh filename=meshes/lipo_battery_mount-v3.stl scale=0.001 0.001 0.001
- added link omni_wheel_mount-v5, mass 0.1235708646349694; collision mesh filename=meshes/omni_wheel_mount-v5.stl scale=0.001 0.001 0.001; visual mesh filename=meshes/omni_wheel_mount-v5.stl scale=0.001 0.001 0.001
- added link omni_wheel_mount-v5-1, mass 0.1235708646349694; collision mesh filename=meshes/omni_wheel_mount-v5-1.stl scale=0.001 0.001 0.001; visual mesh filename=meshes/omni_wheel_mount-v5-1.stl scale=0.001 0.001 0.001
- added link omni_wheel_mount-v5-2, mass 0.1235708646349694; collision mesh filename=meshes/omni_wheel_mount-v5-2.stl scale=0.001 0.001 0.001; visual mesh filename=meshes/omni_wheel_mount-v5-2.stl scale=0.001 0.001 0.001
- added link servo_controller_mount-v3, mass 0.12559881449596652; collision mesh filename=meshes/servo_controller_mount-v3.stl scale=0.001 0.001 0.001; visual mesh filename=meshes/servo_controller_mount-v3.stl scale=0.001 0.001 0.001
Joints:
- removed joint arm_base_joint
- removed joint back_wheel
- removed joint elbow_flex
- removed joint gripper
- removed joint left_wheel
- removed joint right_wheel
- removed joint shoulder_lift
- removed joint shoulder_pan
- removed joint wrist_flex
- removed joint wrist_roll
- added joint 94868A713_NO-THREADS_Female-Threaded-Hex-Standoff_Rigid-21: type fixed, parent 94868A713_NO-THREADS_Female-Threaded-Hex-Standoff, child base_plate_layer2-v3, origin xyz=0.0 0.0 -0.05 rpy=3.141592653589793 -0.0 0.0
- added joint Base_08q-v1_Rigid-43: type fixed, parent Base_08q-v1, child WaveShare_Mounting_Plate_01d-v1, origin xyz=-0.04 -0.07525199 0.060300000000000006 rpy=3.141592653589793 6.259293778842913e-51 2.356194490192345
- added joint Base_08q-v1_Rigid-44: type fixed, parent Base_08q-v1, child STS3215_03a-v1, origin xyz=-0.029750000000000002 -0.045651989999999996 0.027800000000000002 rpy=1.5707963267948966 -8.851978152917189e-51 -2.4803256509655576e-48
- added joint Base_08q-v1_Rigid-47: type fixed, parent Base_08q-v1, child Passive_Horn_01-v1, origin xyz=-0.04 -0.012851990000000004 0.013599999999999994 rpy=-1.5707963267948966 -8.851978152917189e-51 -2.4803256509655576e-48
- added joint Bottom-V2-v3_Rigid-24: type fixed, parent Bottom-V2-v3, child Top-V2-v2, origin xyz=0.0197 0.036125 0.0025 rpy=0.0 -0.0 -2.465190328815662e-32
- added joint Camera-Mount-v8_Rigid-29: type fixed, parent Camera-Mount-v8, child Camera-Model-v3, origin xyz=-0.034 0.00636666 0.03831948 rpy=3.141592653589793 -1.3962634015954636 3.141592653589793
- added joint Rotation_Pitch_08i-v1_Rigid-46: type fixed, parent Rotation_Pitch_08i-v1, child SO_ARM100_08k_Asym_Mirror_Clip-v1, origin xyz=0.023000000000000066 -0.04085 -0.023200000000000002 rpy=-3.944304526105059e-31 -4.116117285135399e-31 -2.781046729970605e-32
- added joint Rotation_Pitch_08i-v1_Rigid-48: type fixed, parent Rotation_Pitch_08i-v1, child STS3215_03a-v1-1, origin xyz=-0.016299999999999943 -0.04085 -0.019400000000000014 rpy=1.8260247115545314e-16 -4.116117285135399e-31 -2.781046729970605e-32
- added joint SO_ARM100_08k_116_Square-v1_Rigid-50: type fixed, parent SO_ARM100_08k_116_Square-v1, child STS3215_03a-v1-2, origin xyz=-0.03610000000000001 -0.10151227 -0.013699510000000003 rpy=-7.511797348558594e-34 -4.930380657631324e-32 1.3877787807814457e-17
- added joint SO_ARM100_08k_Mirror-v1_Rigid-52: type fixed, parent SO_ARM100_08k_Mirror-v1, child STS3215_03a-v1-3, origin xyz=-0.0361 0.09885064 0.03311837999999998 rpy=-3.1415926535897922 5.9164567891575885e-31 2.91703841149741e-62
- added joint ST3215_Servo_Motor-v1-1_Revolute-62: type continuous, parent ST3215_Servo_Motor-v1-1, child omni_wheel_mount-v5-1, origin xyz=0.010249999999999999 0.04636234 -0.014801910000000005 rpy=-1.5707963267948966 1.5707963267948966 0, axis 0.866025 1.0674582272562919e-32 0.5
- added joint ST3215_Servo_Motor-v1-2_Revolute-60: type continuous, parent ST3215_Servo_Motor-v1-2, child omni_wheel_mount-v5-2, origin xyz=0.010249999999999999 -0.035199999999999995 -0.03275 rpy=-1.5707963267948966 1.5707963267948966 0, axis 0.0 0.0 -1.0
- added joint ST3215_Servo_Motor-v1_Revolute-64: type continuous, parent ST3215_Servo_Motor-v1, child omni_wheel_mount-v5, origin xyz=0.010249999999999999 -0.010762340000000004 0.046859090000000006 rpy=-1.5707963267948966 1.5707963267948966 0, axis -0.866025 -2.0578792567370943e-32 0.5
- added joint STS3215_03a-v1-1_Revolute-49: type continuous, parent STS3215_03a-v1-1, child SO_ARM100_08k_116_Square-v1, origin xyz=0.0346 0.010249999999999987 -0.032799999999999975 rpy=3.141592653589793 1.7181275903033976e-32 -3.1373434374976504e-48, axis 1.0 0.0 0.0
- added joint STS3215_03a-v1-2_Revolute-51: type continuous, parent STS3215_03a-v1-2, child SO_ARM100_08k_Mirror-v1, origin xyz=0.0346 -0.013069710000000002 0.03178184000000002 rpy=-6.842277657836021e-49 -3.4512664603419266e-31 -1.3877787807814457e-17, axis 1.0 0.0 0.0
- added joint STS3215_03a-v1-3_Revolute-53: type continuous, parent STS3215_03a-v1-3, child Wrist_Roll_Pitch_08i-v1, origin xyz=0.0346 -0.03408158 0.004398620000000015 rpy=3.1415926535897922 9.860761315262648e-32 -9.503163413661107e-47, axis 1.0 0.0 9.860761315262648e-32
- added joint STS3215_03a-v1-4_Revolute-57: type continuous, parent STS3215_03a-v1-4, child Moving_Jaw_08d-v1, origin xyz=-0.032799999999999996 -0.023912249999999986 0.027026410000000018 rpy=-1.5707963267948968 3.944304526105059e-31 -1.9721522630525295e-31, axis -2.74128770133849e-31 -0.9063079999999999 -0.422618
- added joint STS3215_03a-v1_Revolute-45: type continuous, parent STS3215_03a-v1, child Rotation_Pitch_08i-v1, origin xyz=-0.010250000000000084 0.03459999999999999 -0.032799999999999996 rpy=1.5707963267948966 -2.781046729970605e-32 3.94430452610506e-31, axis -3.944304526105059e-31 3.944304526105059e-31 1.0
- added joint STS3215_03a_Wrist_Roll-v1_Revolute-55: type continuous, parent STS3215_03a_Wrist_Roll-v1, child Wrist_Roll_08c-v1, origin xyz=-0.028999999999999998 0.00810632 0.006869499999999995 rpy=3.141592653589793 -0.0 0.0, axis 0.0 0.42261799999999994 -0.9063079999999999
- added joint Wrist-Camera-Mount-v11_Rigid-71: type fixed, parent Wrist-Camera-Mount-v11, child Camera-Model-v3-1, origin xyz=0.0015500000000000004 0.00712333000000001 0.06397354 rpy=1.5707963267948966 -0.0 2.181661564992912
- added joint Wrist_Roll_08c-v1_Rigid-56: type fixed, parent Wrist_Roll_08c-v1, child STS3215_03a-v1-4, origin xyz=0.012999999999999998 0.019942129999999985 -0.004906820000000014 rpy=1.5707963267948966 -0.0 0.0
- added joint Wrist_Roll_08c-v1_Rigid-58: type fixed, parent Wrist_Roll_08c-v1, child Wrist-Camera-Mount-v11, origin xyz=0.012999999999999998 0.027192599999999983 -0.0015258700000000047 rpy=-1.5707963267948966 -0.0 0.0
- added joint Wrist_Roll_Pitch_08i-v1_Rigid-54: type fixed, parent Wrist_Roll_Pitch_08i-v1, child STS3215_03a_Wrist_Roll-v1, origin xyz=0.0089 0.0339283 -0.04850591000000001 rpy=-3.141592653589793 -9.860761315262648e-32 0.0
- added joint base_plate_layer1-v5_Rigid-15: type fixed, parent base_plate_layer1-v5, child servo_controller_mount-v3, origin xyz=0.0 0.06 0.0 rpy=0.0 -0.0 0.0
- added joint base_plate_layer1-v5_Rigid-18: type fixed, parent base_plate_layer1-v5, child lipo_battery_mount-v3, origin xyz=-0.04 -0.02 0.0 rpy=3.141592653589793 -0.0 0.0
- added joint base_plate_layer1-v5_Rigid-20: type fixed, parent base_plate_layer1-v5, child 94868A713_NO-THREADS_Female-Threaded-Hex-Standoff, origin xyz=0.0 0.0 0.0 rpy=3.141592653589793 -0.0 0.0
- added joint base_plate_layer1-v5_Rigid-28: type fixed, parent base_plate_layer1-v5, child Camera-Mount-v8, origin xyz=0.02 0.1 0.0 rpy=0.0 -0.0 0.0
- added joint base_plate_layer1-v5_Rigid-30: type fixed, parent base_plate_layer1-v5, child 94868A713_NO-THREADS_Female-Threaded-Hex-Standoff-5, origin xyz=0.02 -0.1 0.0 rpy=3.141592653589793 -0.0 0.0
- added joint base_plate_layer1-v5_Rigid-31: type fixed, parent base_plate_layer1-v5, child 94868A713_NO-THREADS_Female-Threaded-Hex-Standoff-4, origin xyz=0.07660254 0.06732051 0.0 rpy=3.141592653589793 -0.0 0.0
- added joint base_plate_layer1-v5_Rigid-32: type fixed, parent base_plate_layer1-v5, child 94868A713_NO-THREADS_Female-Threaded-Hex-Standoff-3, origin xyz=-0.09660254 0.032679490000000005 0.0 rpy=3.141592653589793 -0.0 0.0
- added joint base_plate_layer1-v5_Rigid-69: type fixed, parent base_plate_layer1-v5, child 94868A713_NO-THREADS_Female-Threaded-Hex-Standoff-2, origin xyz=0.1 -0.02 0.0 rpy=3.141592653589793 -0.0 0.0
- added joint base_plate_layer1-v5_Rigid-70: type fixed, parent base_plate_layer1-v5, child 94868A713_NO-THREADS_Female-Threaded-Hex-Standoff-1, origin xyz=-0.1 -0.02 0.0 rpy=3.141592653589793 -0.0 0.0
- added joint base_plate_layer1-v5_baseplate2bottom_mount: type fixed, parent base_plate_layer1-v5, child drive_motor_mount-v11-2, origin xyz=-0.02 -0.1 0.0 rpy=3.141592653589793 -0.0 0.0
- added joint base_plate_layer1-v5_baseplate2left_mount: type fixed, parent base_plate_layer1-v5, child drive_motor_mount-v11, origin xyz=-0.05928203 0.057320510000000005 0.0 rpy=3.141592653589793 -0.0 0.0
- added joint base_plate_layer1-v5_baseplate2right_mount: type fixed, parent base_plate_layer1-v5, child drive_motor_mount-v11-1, origin xyz=0.07928203 0.022679490000000004 0.0 rpy=0.0 -0.0 0.0
- added joint base_plate_layer2-v3_Rigid-22: type fixed, parent base_plate_layer2-v3, child Bottom-V2-v3, origin xyz=-0.02 -0.1 0.007000000000000002 rpy=0.0 -0.0 0.0
- added joint base_plate_layer2-v3_Rigid-42: type fixed, parent base_plate_layer2-v3, child Base_08q-v1, origin xyz=0.04 0.08 0.007000000000000002 rpy=0.0 -0.0 0.0
- added joint drive_motor_mount-v11-1_Rigid-35: type fixed, parent drive_motor_mount-v11-1, child ST3215_Servo_Motor-v1-1, origin xyz=-0.007786400000000002 -0.018513550000000004 0.0076100000000000004 rpy=-7.401486830834375e-17 -1.5707963267948966 0
- added joint drive_motor_mount-v11-2_Rigid-2: type fixed, parent drive_motor_mount-v11-2, child ST3215_Servo_Motor-v1-2, origin xyz=-0.01214 -0.015999999999999997 -0.0076100000000000004 rpy=3.141592653589793 1.5707963267948966 0
- added joint drive_motor_mount-v11_Rigid-39: type fixed, parent drive_motor_mount-v11, child ST3215_Servo_Motor-v1, origin xyz=0.019926399999999997 -0.0025135499999999933 -0.0076100000000000004 rpy=3.141592653589793 1.5707963267948966 0
- added joint lipo_battery_mount-v3_Rigid-19: type fixed, parent lipo_battery_mount-v3, child Battery---Battery-5.2-Ah-DC5521-Plug-v2, origin xyz=-0.011500000000000003 0.0 -0.006500000000000001 rpy=3.141592653589793 -0.0 0.0
- added joint omni_wheel_mount-v5-1_Rigid-63: type fixed, parent omni_wheel_mount-v5-1, child 4-Omni-Directional-Wheel_Single_Body-v1-1, origin xyz=0.0062137300000000015 0.0 0.0035875000000000056 rpy=-1.5707963267948966 5.551115123125765e-17 -1.8816263559048997e-48
- added joint omni_wheel_mount-v5-2_Rigid-61: type fixed, parent omni_wheel_mount-v5-2, child 4-Omni-Directional-Wheel_Single_Body-v1-2, origin xyz=0.0 0.0 -0.007174999999999994 rpy=-1.5707963267948966 -0.0 0.0
- added joint omni_wheel_mount-v5_Rigid-65: type fixed, parent omni_wheel_mount-v5, child 4-Omni-Directional-Wheel_Single_Body-v1, origin xyz=-0.0062137300000000015 0.0 0.003587499999999997 rpy=-1.5707963267948966 5.551115123125802e-17 4.930380657631324e-32
