Commit message: chore: apply code review feedback

File: packages/physicalai-lekiwi-plugin/urdf/lekiwi/urdf/LeKiwi.urdf (robot description, URDF)
Before this commit: robot LeKiwi, 45 links, 44 joints
Links:
- link 4-Omni-Directional-Wheel_Single_Body-v1: geometry collision mesh filename=../meshes/4-Omni-Directional-Wheel_Single_Body-v1.stl scale=0.001 0.001 0.001; visual mesh filename=../meshes/4-Omni-Directional-Wheel_Single_Body-v1.stl scale=0.001 0.001 0.001
- link 4-Omni-Directional-Wheel_Single_Body-v1-1: geometry collision mesh filename=../meshes/4-Omni-Directional-Wheel_Single_Body-v1-1.stl scale=0.001 0.001 0.001; visual mesh filename=../meshes/4-Omni-Directional-Wheel_Single_Body-v1-1.stl scale=0.001 0.001 0.001
- link 4-Omni-Directional-Wheel_Single_Body-v1-2: geometry collision mesh filename=../meshes/4-Omni-Directional-Wheel_Single_Body-v1-2.stl scale=0.001 0.001 0.001; visual mesh filename=../meshes/4-Omni-Directional-Wheel_Single_Body-v1-2.stl scale=0.001 0.001 0.001
- link 94868A713_NO-THREADS_Female-Threaded-Hex-Standoff: geometry collision mesh filename=../meshes/94868A713_NO-THREADS_Female-Threaded-Hex-Standoff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 scale=0.001 0.001 0.001; visual mesh filename=../meshes/94868A713_NO-THREADS_Female-Threaded-Hex-Standoff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 scale=0.001 0.001 0.001
- link 94868A713_NO-THREADS_Female-Threaded-Hex-Standoff-1: geometry collision mesh filename=../meshes/94868A713_NO-THREADS_Female-Threaded-Hex-Standoff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 scale=0.001 0.001 0.001; visual mesh filename=../meshes/94868A713_NO-THREADS_Female-Threaded-Hex-Standoff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 scale=0.001 0.001 0.001
- link 94868A713_NO-THREADS_Female-Threaded-Hex-Standoff-2: geometry collision mesh filename=../meshes/94868A713_NO-THREADS_Female-Threaded-Hex-Standoff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 scale=0.001 0.001 0.001; visual mesh filename=../meshes/94868A713_NO-THREADS_Female-Threaded-Hex-Standoff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 scale=0.001 0.001 0.001
- link 94868A713_NO-THREADS_Female-Threaded-Hex-Standoff-3: geometry collision mesh filename=../meshes/94868A713_NO-THREADS_Female-Threaded-Hex-Standoff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 scale=0.001 0.001 0.001; visual mesh filename=../meshes/94868A713_NO-THREADS_Female-Threaded-Hex-Standoff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 scale=0.001 0.001 0.001
- link 94868A713_NO-THREADS_Female-Threaded-Hex-Standoff-4: geometry collision mesh filename=../meshes/94868A713_NO-THREADS_Female-Threaded-Hex-Standoff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 scale=0.001 0.001 0.001; visual mesh filename=../meshes/94868A713_NO-THREADS_Female-Threaded-Hex-Standoff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 scale=0.001 0.001 0.001
- link 94868A713_NO-THREADS_Female-Threaded-Hex-Standoff-5: geometry collision mesh filename=../meshes/94868A713_NO-THREADS_Female-Threaded-Hex-Standoff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 scale=0.001 0.001 0.001; visual mesh filename=../meshes/94868A713_NO-THREADS_Female-Threaded-Hex-Standoff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 scale=0.001 0.001 0.001
- link Base_08q-v1: geometry collision mesh filename=../meshes/Base_08q-v1.stl scale=0.001 0.001 0.001; visual mesh filename=../meshes/Base_08q-v1.stl scale=0.001 0.001 0.001
- link Battery---Battery-5.2-Ah-DC5521-Plug-v2: geometry collision mesh filename=../meshes/Battery---Battery-5.2-Ah-DC5521-Plug-v2.stl scale=0.001 0.001 0.001; visual mesh filename=../meshes/Battery---Battery-5.2-Ah-DC5521-Plug-v2.stl scale=0.001 0.001 0.001
- link Bottom-V2-v3: geometry collision mesh filename=../meshes/Bottom-V2-v3.stl scale=0.001 0.001 0.001; visual mesh filename=../meshes/Bottom-V2-v3.stl scale=0.001 0.001 0.001
- link Camera-Model-v3: geometry collision mesh filename=../meshes/Camera-Model-v3.stl scale=0.001 0.001 0.001; visual mesh filename=../meshes/Camera-Model-v3.stl scale=0.001 0.001 0.001
- link Camera-Model-v3-1: geometry collision mesh filename=../meshes/Camera-Model-v3-1.stl scale=0.001 0.001 0.001; visual mesh filename=../meshes/Camera-Model-v3-1.stl scale=0.001 0.001 0.001
- link Camera-Mount-v8: geometry collision mesh filename=../meshes/Camera-Mount-v8.stl scale=0.001 0.001 0.001; visual mesh filename=../meshes/Camera-Mount-v8.stl scale=0.001 0.001 0.001
- link Moving_Jaw_08d-v1: geometry collision mesh filename=../meshes/Moving_Jaw_08d-v1.stl scale=0.001 0.001 0.001; visual mesh filename=../meshes/Moving_Jaw_08d-v1.stl scale=0.001 0.001 0.001
- link Passive_Horn_01-v1: geometry collision mesh filename=../meshes/Passive_Horn_01-v1.stl scale=0.001 0.001 0.001; visual mesh filename=../meshes/Passive_Horn_01-v1.stl scale=0.001 0.001 0.001
- link Rotation_Pitch_08i-v1: geometry collision mesh filename=../meshes/Rotation_Pitch_08i-v1.stl scale=0.001 0.001 0.001; visual mesh filename=../meshes/Rotation_Pitch_08i-v1.stl scale=0.001 0.001 0.001
- link SO_ARM100_08k_116_Square-v1: geometry collision mesh filename=../meshes/SO_ARM100_08k_116_Square-v1.stl scale=0.001 0.001 0.001; visual mesh filename=../meshes/SO_ARM100_08k_116_Square-v1.stl scale=0.001 0.001 0.001
- link SO_ARM100_08k_Asym_Mirror_Clip-v1: geometry collision mesh filename=../meshes/SO_ARM100_08k_Asym_Mirror_Clip-v1.stl scale=0.001 0.001 0.001; visual mesh filename=../meshes/SO_ARM100_08k_Asym_Mirror_Clip-v1.stl scale=0.001 0.001 0.001
- link SO_ARM100_08k_Mirror-v1: geometry collision mesh filename=../meshes/SO_ARM100_08k_Mirror-v1.stl scale=0.001 0.001 0.001; visual mesh filename=../meshes/SO_ARM100_08k_Mirror-v1.stl scale=0.001 0.001 0.001
- link ST3215_Servo_Motor-v1: geometry collision mesh filename=../meshes/ST3215_Servo_Motor-v1.stl scale=0.001 0.001 0.001; visual mesh filename=../meshes/ST3215_Servo_Motor-v1.stl scale=0.001 0.001 0.001
- link ST3215_Servo_Motor-v1-1: geometry collision mesh filename=../meshes/ST3215_Servo_Motor-v1-1.stl scale=0.001 0.001 0.001; visual mesh filename=../meshes/ST3215_Servo_Motor-v1-1.stl scale=0.001 0.001 0.001
- link ST3215_Servo_Motor-v1-2: geometry collision mesh filename=../meshes/ST3215_Servo_Motor-v1-2.stl scale=0.001 0.001 0.001; visual mesh filename=../meshes/ST3215_Servo_Motor-v1-2.stl scale=0.001 0.001 0.001
- link STS3215_03a-v1: geometry collision mesh filename=../meshes/STS3215_03a-v1.stl scale=0.001 0.001 0.001; visual mesh filename=../meshes/STS3215_03a-v1.stl scale=0.001 0.001 0.001
- link STS3215_03a-v1-1: geometry collision mesh filename=../meshes/STS3215_03a-v1-1.stl scale=0.001 0.001 0.001; visual mesh filename=../meshes/STS3215_03a-v1-1.stl scale=0.001 0.001 0.001
- link STS3215_03a-v1-2: geometry collision mesh filename=../meshes/STS3215_03a-v1-2.stl scale=0.001 0.001 0.001; visual mesh filename=../meshes/STS3215_03a-v1-2.stl scale=0.001 0.001 0.001
- link STS3215_03a-v1-3: geometry collision mesh filename=../meshes/STS3215_03a-v1-3.stl scale=0.001 0.001 0.001; visual mesh filename=../meshes/STS3215_03a-v1-3.stl scale=0.001 0.001 0.001
- link STS3215_03a-v1-4: geometry collision mesh filename=../meshes/STS3215_03a-v1-4.stl scale=0.001 0.001 0.001; visual mesh filename=../meshes/STS3215_03a-v1-4.stl scale=0.001 0.001 0.001
- link STS3215_03a_Wrist_Roll-v1: geometry collision mesh filename=../meshes/STS3215_03a_Wrist_Roll-v1.stl scale=0.001 0.001 0.001; visual mesh filename=../meshes/STS3215_03a_Wrist_Roll-v1.stl scale=0.001 0.001 0.001
- link Top-V2-v2: geometry collision mesh filename=../meshes/Top-V2-v2.stl scale=0.001 0.001 0.001; visual mesh filename=../meshes/Top-V2-v2.stl scale=0.001 0.001 0.001
- link WaveShare_Mounting_Plate_01d-v1: geometry collision mesh filename=../meshes/WaveShare_Mounting_Plate_01d-v1.stl scale=0.001 0.001 0.001; visual mesh filename=../meshes/WaveShare_Mounting_Plate_01d-v1.stl scale=0.001 0.001 0.001
- link Wrist-Camera-Mount-v11: geometry collision mesh filename=../meshes/Wrist-Camera-Mount-v11.stl scale=0.001 0.001 0.001; visual mesh filename=../meshes/Wrist-Camera-Mount-v11.stl scale=0.001 0.001 0.001
- link Wrist_Roll_08c-v1: geometry collision mesh filename=../meshes/Wrist_Roll_08c-v1.stl scale=0.001 0.001 0.001; visual mesh filename=../meshes/Wrist_Roll_08c-v1.stl scale=0.001 0.001 0.001
- link Wrist_Roll_Pitch_08i-v1: geometry collision mesh filename=../meshes/Wrist_Roll_Pitch_08i-v1.stl scale=0.001 0.001 0.001; visual mesh filename=../meshes/Wrist_Roll_Pitch_08i-v1.stl scale=0.001 0.001 0.001
- link base_plate_layer1-v5: geometry collision mesh filename=../meshes/base_plate_layer1-v5.stl scale=0.001 0.001 0.001; visual mesh filename=../meshes/base_plate_layer1-v5.stl scale=0.001 0.001 0.001
- link base_plate_layer2-v3: geometry collision mesh filename=../meshes/base_plate_layer2-v3.stl scale=0.001 0.001 0.001; visual mesh filename=../meshes/base_plate_layer2-v3.stl scale=0.001 0.001 0.001
- link drive_motor_mount-v11: geometry collision mesh filename=../meshes/drive_motor_mount-v11.stl scale=0.001 0.001 0.001; visual mesh filename=../meshes/drive_motor_mount-v11.stl scale=0.001 0.001 0.001
- link drive_motor_mount-v11-1: geometry collision mesh filename=../meshes/drive_motor_mount-v11-1.stl scale=0.001 0.001 0.001; visual mesh filename=../meshes/drive_motor_mount-v11-1.stl scale=0.001 0.001 0.001
- link drive_motor_mount-v11-2: geometry collision mesh filename=../meshes/drive_motor_mount-v11-2.stl scale=0.001 0.001 0.001; visual mesh filename=../meshes/drive_motor_mount-v11-2.stl scale=0.001 0.001 0.001
- link lipo_battery_mount-v3: geometry collision mesh filename=../meshes/lipo_battery_mount-v3.stl scale=0.001 0.001 0.001; visual mesh filename=../meshes/lipo_battery_mount-v3.stl scale=0.001 0.001 0.001
- link omni_wheel_mount-v5: geometry collision mesh filename=../meshes/omni_wheel_mount-v5.stl scale=0.001 0.001 0.001; visual mesh filename=../meshes/omni_wheel_mount-v5.stl scale=0.001 0.001 0.001
- link omni_wheel_mount-v5-1: geometry collision mesh filename=../meshes/omni_wheel_mount-v5-1.stl scale=0.001 0.001 0.001; visual mesh filename=../meshes/omni_wheel_mount-v5-1.stl scale=0.001 0.001 0.001
- link omni_wheel_mount-v5-2: geometry collision mesh filename=../meshes/omni_wheel_mount-v5-2.stl scale=0.001 0.001 0.001; visual mesh filename=../meshes/omni_wheel_mount-v5-2.stl scale=0.001 0.001 0.001
- link servo_controller_mount-v3: geometry collision mesh filename=../meshes/servo_controller_mount-v3.stl scale=0.001 0.001 0.001; visual mesh filename=../meshes/servo_controller_mount-v3.stl scale=0.001 0.001 0.001

Commit message: fix: fix path to lekiwi meshes

File: packages/physicalai-lekiwi-plugin/urdf/lekiwi/urdf/LeKiwi.urdf (robot description, URDF)
Before this commit: robot LeKiwi, 45 links, 44 joints
Links:
- link 4-Omni-Directional-Wheel_Single_Body-v1: geometry collision mesh filename=meshes/4-Omni-Directional-Wheel_Single_Body-v1.stl scale=0.001 0.001 0.001; visual mesh filename=meshes/4-Omni-Directional-Wheel_Single_Body-v1.stl scale=0.001 0.001 0.001
- link 4-Omni-Directional-Wheel_Single_Body-v1-1: geometry collision mesh filename=meshes/4-Omni-Directional-Wheel_Single_Body-v1-1.stl scale=0.001 0.001 0.001; visual mesh filename=meshes/4-Omni-Directional-Wheel_Single_Body-v1-1.stl scale=0.001 0.001 0.001
- link 4-Omni-Directional-Wheel_Single_Body-v1-2: geometry collision mesh filename=meshes/4-Omni-Directional-Wheel_Single_Body-v1-2.stl scale=0.001 0.001 0.001; visual mesh filename=meshes/4-Omni-Directional-Wheel_Single_Body-v1-2.stl scale=0.001 0.001 0.001
- link 94868A713_NO-THREADS_Female-Threaded-Hex-Standoff: geometry collision mesh filename=meshes/94868A713_NO-THREADS_Female-Threaded-Hex-Standoff.stl scale=0.001 0.001 0.001; visual mesh filename=meshes/94868A713_NO-THREADS_Female-Threaded-Hex-Standoff.stl scale=0.001 0.001 0.001
- link 94868A713_NO-THREADS_Female-Threaded-Hex-Standoff-1: geometry collision mesh filename=meshes/94868A713_NO-THREADS_Female-Threaded-Hex-Standoff-1.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 scale=0.001 0.001 0.001; visual mesh filename=meshes/94868A713_NO-THREADS_Female-Threaded-Hex-Standoff-1.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 scale=0.001 0.001 0.001
- link 94868A713_NO-THREADS_Female-Threaded-Hex-Standoff-2: geometry collision mesh filename=meshes/94868A713_NO-THREADS_Female-Threaded-Hex-Standoff-2.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 scale=0.001 0.001 0.001; visual mesh filename=meshes/94868A713_NO-THREADS_Female-Threaded-Hex-Standoff-2.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 scale=0.001 0.001 0.001
- link 94868A713_NO-THREADS_Female-Threaded-Hex-Standoff-3: geometry collision mesh filename=meshes/94868A713_NO-THREADS_Female-Threaded-Hex-Standoff-3.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 scale=0.001 0.001 0.001; visual mesh filename=meshes/94868A713_NO-THREADS_Female-Threaded-Hex-Standoff-3.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 scale=0.001 0.001 0.001
- link 94868A713_NO-THREADS_Female-Threaded-Hex-Standoff-4: geometry collision mesh filename=meshes/94868A713_NO-THREADS_Female-Threaded-Hex-Standoff-4.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 scale=0.001 0.001 0.001; visual mesh filename=meshes/94868A713_NO-THREADS_Female-Threaded-Hex-Standoff-4.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 scale=0.001 0.001 0.001
- link 94868A713_NO-THREADS_Female-Threaded-Hex-Standoff-5: geometry collision mesh filename=meshes/94868A713_NO-THREADS_Female-Threaded-Hex-Standoff-5.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 scale=0.001 0.001 0.001; visual mesh filename=meshes/94868A713_NO-THREADS_Female-Threaded-Hex-Standoff-5.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 scale=0.001 0.001 0.001
- link Base_08q-v1: geometry collision mesh filename=meshes/Base_08q-v1.stl scale=0.001 0.001 0.001; visual mesh filename=meshes/Base_08q-v1.stl scale=0.001 0.001 0.001
- link Battery---Battery-5.2-Ah-DC5521-Plug-v2: geometry collision mesh filename=meshes/Battery---Battery-5.2-Ah-DC5521-Plug-v2.stl scale=0.001 0.001 0.001; visual mesh filename=meshes/Battery---Battery-5.2-Ah-DC5521-Plug-v2.stl scale=0.001 0.001 0.001
- link Bottom-V2-v3: geometry collision mesh filename=meshes/Bottom-V2-v3.stl scale=0.001 0.001 0.001; visual mesh filename=meshes/Bottom-V2-v3.stl scale=0.001 0.001 0.001
- link Camera-Model-v3: geometry collision mesh filename=meshes/Camera-Model-v3.stl scale=0.001 0.001 0.001; visual mesh filename=meshes/Camera-Model-v3.stl scale=0.001 0.001 0.001
- link Camera-Model-v3-1: geometry collision mesh filename=meshes/Camera-Model-v3-1.stl scale=0.001 0.001 0.001; visual mesh filename=meshes/Camera-Model-v3-1.stl scale=0.001 0.001 0.001
- link Camera-Mount-v8: geometry collision mesh filename=meshes/Camera-Mount-v8.stl scale=0.001 0.001 0.001; visual mesh filename=meshes/Camera-Mount-v8.stl scale=0.001 0.001 0.001
- link Moving_Jaw_08d-v1: geometry collision mesh filename=meshes/Moving_Jaw_08d-v1.stl scale=0.001 0.001 0.001; visual mesh filename=meshes/Moving_Jaw_08d-v1.stl scale=0.001 0.001 0.001
- link Passive_Horn_01-v1: geometry collision mesh filename=meshes/Passive_Horn_01-v1.stl scale=0.001 0.001 0.001; visual mesh filename=meshes/Passive_Horn_01-v1.stl scale=0.001 0.001 0.001
- link Rotation_Pitch_08i-v1: geometry collision mesh filename=meshes/Rotation_Pitch_08i-v1.stl scale=0.001 0.001 0.001; visual mesh filename=meshes/Rotation_Pitch_08i-v1.stl scale=0.001 0.001 0.001
- link SO_ARM100_08k_116_Square-v1: geometry collision mesh filename=meshes/SO_ARM100_08k_116_Square-v1.stl scale=0.001 0.001 0.001; visual mesh filename=meshes/SO_ARM100_08k_116_Square-v1.stl scale=0.001 0.001 0.001
- link SO_ARM100_08k_Asym_Mirror_Clip-v1: geometry collision mesh filename=meshes/SO_ARM100_08k_Asym_Mirror_Clip-v1.stl scale=0.001 0.001 0.001; visual mesh filename=meshes/SO_ARM100_08k_Asym_Mirror_Clip-v1.stl scale=0.001 0.001 0.001
- link SO_ARM100_08k_Mirror-v1: geometry collision mesh filename=meshes/SO_ARM100_08k_Mirror-v1.stl scale=0.001 0.001 0.001; visual mesh filename=meshes/SO_ARM100_08k_Mirror-v1.stl scale=0.001 0.001 0.001
- link ST3215_Servo_Motor-v1: geometry collision mesh filename=meshes/ST3215_Servo_Motor-v1.stl scale=0.001 0.001 0.001; visual mesh filename=meshes/ST3215_Servo_Motor-v1.stl scale=0.001 0.001 0.001
- link ST3215_Servo_Motor-v1-1: geometry collision mesh filename=meshes/ST3215_Servo_Motor-v1-1.stl scale=0.001 0.001 0.001; visual mesh filename=meshes/ST3215_Servo_Motor-v1-1.stl scale=0.001 0.001 0.001
- link ST3215_Servo_Motor-v1-2: geometry collision mesh filename=meshes/ST3215_Servo_Motor-v1-2.stl scale=0.001 0.001 0.001; visual mesh filename=meshes/ST3215_Servo_Motor-v1-2.stl scale=0.001 0.001 0.001
- link STS3215_03a-v1: geometry collision mesh filename=meshes/STS3215_03a-v1.stl scale=0.001 0.001 0.001; visual mesh filename=meshes/STS3215_03a-v1.stl scale=0.001 0.001 0.001
- link STS3215_03a-v1-1: geometry collision mesh filename=meshes/STS3215_03a-v1-1.stl scale=0.001 0.001 0.001; visual mesh filename=meshes/STS3215_03a-v1-1.stl scale=0.001 0.001 0.001
- link STS3215_03a-v1-2: geometry collision mesh filename=meshes/STS3215_03a-v1-2.stl scale=0.001 0.001 0.001; visual mesh filename=meshes/STS3215_03a-v1-2.stl scale=0.001 0.001 0.001
- link STS3215_03a-v1-3: geometry collision mesh filename=meshes/STS3215_03a-v1-3.stl scale=0.001 0.001 0.001; visual mesh filename=meshes/STS3215_03a-v1-3.stl scale=0.001 0.001 0.001
- link STS3215_03a-v1-4: geometry collision mesh filename=meshes/STS3215_03a-v1-4.stl scale=0.001 0.001 0.001; visual mesh filename=meshes/STS3215_03a-v1-4.stl scale=0.001 0.001 0.001
- link STS3215_03a_Wrist_Roll-v1: geometry collision mesh filename=meshes/STS3215_03a_Wrist_Roll-v1.stl scale=0.001 0.001 0.001; visual mesh filename=meshes/STS3215_03a_Wrist_Roll-v1.stl scale=0.001 0.001 0.001
- link Top-V2-v2: geometry collision mesh filename=meshes/Top-V2-v2.stl scale=0.001 0.001 0.001; visual mesh filename=meshes/Top-V2-v2.stl scale=0.001 0.001 0.001
- link WaveShare_Mounting_Plate_01d-v1: geometry collision mesh filename=meshes/WaveShare_Mounting_Plate_01d-v1.stl scale=0.001 0.001 0.001; visual mesh filename=meshes/WaveShare_Mounting_Plate_01d-v1.stl scale=0.001 0.001 0.001
- link Wrist-Camera-Mount-v11: geometry collision mesh filename=meshes/Wrist-Camera-Mount-v11.stl scale=0.001 0.001 0.001; visual mesh filename=meshes/Wrist-Camera-Mount-v11.stl scale=0.001 0.001 0.001
- link Wrist_Roll_08c-v1: geometry collision mesh filename=meshes/Wrist_Roll_08c-v1.stl scale=0.001 0.001 0.001; visual mesh filename=meshes/Wrist_Roll_08c-v1.stl scale=0.001 0.001 0.001
- link Wrist_Roll_Pitch_08i-v1: geometry collision mesh filename=meshes/Wrist_Roll_Pitch_08i-v1.stl scale=0.001 0.001 0.001; visual mesh filename=meshes/Wrist_Roll_Pitch_08i-v1.stl scale=0.001 0.001 0.001
- link base_plate_layer1-v5: geometry collision mesh filename=meshes/base_plate_layer1-v5.stl scale=0.001 0.001 0.001; visual mesh filename=meshes/base_plate_layer1-v5.stl scale=0.001 0.001 0.001
- link base_plate_layer2-v3: geometry collision mesh filename=meshes/base_plate_layer2-v3.stl scale=0.001 0.001 0.001; visual mesh filename=meshes/base_plate_layer2-v3.stl scale=0.001 0.001 0.001
- link drive_motor_mount-v11: geometry collision mesh filename=meshes/drive_motor_mount-v11.stl scale=0.001 0.001 0.001; visual mesh filename=meshes/drive_motor_mount-v11.stl scale=0.001 0.001 0.001
- link drive_motor_mount-v11-1: geometry collision mesh filename=meshes/drive_motor_mount-v11-1.stl scale=0.001 0.001 0.001; visual mesh filename=meshes/drive_motor_mount-v11-1.stl scale=0.001 0.001 0.001
- link drive_motor_mount-v11-2: geometry collision mesh filename=meshes/drive_motor_mount-v11-2.stl scale=0.001 0.001 0.001; visual mesh filename=meshes/drive_motor_mount-v11-2.stl scale=0.001 0.001 0.001
- link lipo_battery_mount-v3: geometry collision mesh filename=meshes/lipo_battery_mount-v3.stl scale=0.001 0.001 0.001; visual mesh filename=meshes/lipo_battery_mount-v3.stl scale=0.001 0.001 0.001
- link omni_wheel_mount-v5: geometry collision mesh filename=meshes/omni_wheel_mount-v5.stl scale=0.001 0.001 0.001; visual mesh filename=meshes/omni_wheel_mount-v5.stl scale=0.001 0.001 0.001
- link omni_wheel_mount-v5-1: geometry collision mesh filename=meshes/omni_wheel_mount-v5-1.stl scale=0.001 0.001 0.001; visual mesh filename=meshes/omni_wheel_mount-v5-1.stl scale=0.001 0.001 0.001
- link omni_wheel_mount-v5-2: geometry collision mesh filename=meshes/omni_wheel_mount-v5-2.stl scale=0.001 0.001 0.001; visual mesh filename=meshes/omni_wheel_mount-v5-2.stl scale=0.001 0.001 0.001
- link servo_controller_mount-v3: geometry collision mesh filename=meshes/servo_controller_mount-v3.stl scale=0.001 0.001 0.001; visual mesh filename=meshes/servo_controller_mount-v3.stl scale=0.001 0.001 0.001
