Commit message: fix: resolve lerobot test failures and address review feedback
- Fix cross-package sys.modules pollution: the lekiwi test stubbed
  scservo_sdk without a ModuleSpec, causing importlib.find_spec() to raise
  ValueError when lerobot probes optional SDKs during import
- Suppress false-positive python37 Semgrep rule on importlib.resources
  (package requires Python >=3.12), matching the existing rebot plugin
- Declare pyserial dependency used by studio_catalog serial port probing
- Fix broken README link to the plugin development guide
- Replace placeholder URDF links with a valid revolute-joint chain

File: packages/physicalai-lerobot-plugin/urdf/lerobot/urdf/lerobot.urdf (robot description, URDF)
Before this commit: robot lerobot, 7 links, 0 joints
Links:
- removed link joint1
- removed link joint2
- removed link joint3
- removed link joint4
- removed link joint5
- removed link joint6
- added link link1
- added link link2
- added link link3
- added link link4
- added link link5
- added link link6
Joints:
- added joint joint1: type revolute, parent base_link, child link1, origin xyz=0 0 0 rpy=0 0 0, axis 0 0 1
- added joint joint2: type revolute, parent link1, child link2, origin xyz=0 0 0 rpy=0 0 0, axis 0 0 1
- added joint joint3: type revolute, parent link2, child link3, origin xyz=0 0 0 rpy=0 0 0, axis 0 0 1
- added joint joint4: type revolute, parent link3, child link4, origin xyz=0 0 0 rpy=0 0 0, axis 0 0 1
- added joint joint5: type revolute, parent link4, child link5, origin xyz=0 0 0 rpy=0 0 0, axis 0 0 1
- added joint joint6: type revolute, parent link5, child link6, origin xyz=0 0 0 rpy=0 0 0, axis 0 0 1
