Commit message: chore: colorize rebot and stararm amrs

File: packages/physicalai-rebot-b601-plugin/urdf/rebot-b601-dm/urdf/reBot-DevArm_fixend.urdf (robot description, URDF)
Before this commit: robot reBot-DevArm_fixend, 8 links, 7 joints
Links:
- added link finger_left_link; collision mesh filename=meshes/left_finger.stl; visual mesh filename=meshes/colored_left_finger_carriage_grey.stl
- added link finger_right_link; collision mesh filename=meshes/right_finger.stl; visual mesh filename=meshes/colored_right_finger_carriage_grey.stl
- link base_link: geometry collision mesh filename=meshes/base_link.STL; visual mesh filename=meshes/colored_base_link_hardware_black.stl
- link end_link: mass 0.4500000 -> 0.5000000; geometry collision mesh filename=meshes/gripper_base.stl; visual mesh filename=meshes/colored_gripper_base_hardware_black.stl
- link link1: geometry collision mesh filename=meshes/link1.STL; visual mesh filename=meshes/colored_link1_anodized_grey.stl
- link link2: geometry collision mesh filename=meshes/link2.STL; visual mesh filename=meshes/colored_link2_anodized_grey.stl
- link link3: geometry collision mesh filename=meshes/link3.STL; visual mesh filename=meshes/colored_link3_anodized_grey.stl
- link link4: geometry collision mesh filename=meshes/link4.STL; visual mesh filename=meshes/colored_link4_anodized_grey.stl
- link link5: geometry collision mesh filename=meshes/link5.STL; visual mesh filename=meshes/colored_link5_anodized_grey.stl
- link link6: geometry collision mesh filename=meshes/link6.STL; visual mesh filename=meshes/colored_link6_hardware_black.stl
Joints:
- added joint finger_left: type prismatic, parent end_link, child finger_left_link, origin xyz=0 0 0 rpy=0 0 0, axis 0 1 0, limit lower=0 upper=0.0285 effort=8 velocity=0.08
- added joint finger_right: type prismatic, parent end_link, child finger_right_link, origin xyz=0 0 0 rpy=0 0 0, axis 0 1 0, limit lower=-0.0285 upper=0 effort=8 velocity=0.08, mimic joint=finger_left multiplier=-1 offset=0

File: packages/physicalai-rebot-b601-plugin/urdf/rebot-b601-rs/urdf/00-arm-rs_asm-v3.urdf (robot description, URDF)
Before this commit: robot 00-arm-rs_asm-v3, 10 links, 9 joints
Links:
- link link3: geometry collision mesh filename=meshes/link3.STL; visual mesh filename=meshes/cnc3.STL
Joints:
- removed joint joint_left
- removed joint joint_right
- added joint gripper_joint1: type prismatic, parent gripper_end, child gripper_left, origin xyz=-0.041939 -7.3385E-05 0 rpy=1.5708 -1.5708 0, axis 0 0 1, limit lower=0 upper=0.05 effort=500 velocity=10
- added joint gripper_joint2: type prismatic, parent gripper_end, child gripper_right, origin xyz=-0.041939 7.3385E-05 0 rpy=-1.5708 -1.5708 0, axis 0 0 1, limit lower=0 upper=0.0715 effort=500 velocity=10

File: packages/physicalai-rebot-b601-plugin/urdf/stararm102/urdf/stararm102_description.urdf (robot description, URDF)
Before this commit: robot stararm102_description, 10 links, 9 joints
Links:
- removed link world
- link base_link: geometry collision mesh filename=package://stararm102/meshes/base_link.STL; visual mesh filename=package://stararm102/meshes/shells/base_link__0.STL
- link link1: geometry collision mesh filename=package://stararm102/meshes/link1.STL; visual mesh filename=package://stararm102/meshes/shells/link1__0.STL
- link link2: geometry collision mesh filename=package://stararm102/meshes/link2.STL; visual mesh filename=package://stararm102/meshes/shells/link2__0.STL
- link link3: geometry collision mesh filename=package://stararm102/meshes/link3.STL; visual mesh filename=package://stararm102/meshes/shells/link3__0.STL
- link link4: geometry collision mesh filename=package://stararm102/meshes/link4.STL; visual mesh filename=package://stararm102/meshes/shells/link4__0.STL
- link link5: geometry collision mesh filename=package://stararm102/meshes/link5.STL; visual mesh filename=package://stararm102/meshes/shells/link5__0.STL
- link link6: geometry collision mesh filename=package://stararm102/meshes/link6.STL; visual mesh filename=package://stararm102/meshes/shells/link6__0.STL
- link link7_left: geometry collision mesh filename=package://stararm102/meshes/link7_left.STL; visual mesh filename=package://stararm102/meshes/shells/link7_left__0.STL
- link link7_right: geometry collision mesh filename=package://stararm102/meshes/link7_right.STL; visual mesh filename=package://stararm102/meshes/shells/link7_right__0.STL
Joints:
- removed joint world_to_base
