Commit message: fix: fix lighting and arm position

File: packages/physicalai-openarm-plugin/urdf/openarm_description/openarm_v20_right_arm_pinch.urdf (robot description, URDF)
Before this commit: robot openarm_v20, 11 links, 10 joints
Joints:
- joint openarm_right_base_link_mount_joint: origin xyz=0.0 0.0 0.0 rpy=0.0 0.0 0.0 -> xyz=0.0 0.0 0.605947 rpy=0.0 0.0 0.0
